File: schematic/main.brd (EAGLE design)
At the start: 160 x 100 mm, 38 parts, among them IC1 FT232RL, U1 SI4463-C2A-GM, U2 CG2179M2, U3 STM32L011, X1 SMA

Commit message: Add files via upload
Parts:
- removed R3: 0R, resistor:R0805
- moved CC3 125.3 mm to (65.7, 6.03), turned to 180 degrees
- moved CM3 124.8 mm to (70.5, 11.7), turned to 180 degrees
- moved CC2 123.0 mm to (69.5, 4.45), turned to 90 degrees
- moved U2 122.1 mm to (65.7, 3.49), turned to 270 degrees
- moved CM2 119.6 mm to (69.5, 8.57), turned to 90 degrees
- moved CR1 118.2 mm to (57.8, 7.94), turned to 270 degrees
- moved CM 112.0 mm to (62.2, 12.1), turned to 90 degrees
- moved LR2 111.8 mm to (60.0, 6.67), turned to 270 degrees
- moved LM3 110.5 mm to (71.7, 8.57), turned to 90 degrees
- moved CC1 109.3 mm to (62.2, 5.71), turned to 270 degrees
- moved CM1 108.9 mm to (64.4, 12.1), turned to 90 degrees
- moved C0 102.8 mm to (57.8, 12.1), turned to 90 degrees
- moved LR1 101.0 mm to (55.6, 7.94), turned to 270 degrees
- moved LM2 99.2 mm to (66.7, 9.21), turned to 270 degrees
- moved X1 97.3 mm to (77.0, 9.50), turned to 180 degrees
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Connections:
- removed net N$1: R3.2, U3.31
- net GND: now also U3.31; no longer R3.1
Routing:
- net +3V3: track 14.2 -> 84.4 mm, vias 0 -> 2
- net RX_SW: track 0.00 -> 33.3 mm, vias 0 -> 2
- net TX_SW: track 0.00 -> 32.7 mm, vias 0 -> 2
- net USB_TX: track 0.00 -> 20.5 mm, vias 0 -> 2
- net USB_RX: track 0.00 -> 20.0 mm, vias 0 -> 2
- net SDN: track 0.00 -> 19.8 mm, vias 0 -> 2
- net NRST: track 0.00 -> 14.9 mm, vias 0 -> 1
- net SPI_SCK: track 0.00 -> 11.3 mm, vias 0 -> 2
- net NIRQ: track 0.00 -> 10.5 mm, vias 0 -> 2
- net RF_RXN: track 0.00 -> 7.99 mm
- net SPI_MISO: track 0.00 -> 7.60 mm, vias 0 -> 2
- net NSEL: track 0.00 -> 7.25 mm
- net SPI_MOSI: track 0.00 -> 7.08 mm
- net RF_RXP: track 0.00 -> 6.33 mm
- net SWDIO: track 0.00 -> 6.08 mm
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- added copper zone on layer 1, net GND
- added copper zone on layer 16, net GND
Other:
- board size 160 x 100 mm -> 77 x 19 mm
- board text added: "M17_ANL_1.0"
- board text added: "RF"
- board text added: "SP5WWP"
- board text added: "SWD"
- board text added: "USB"

Commit message: Add files via upload
Connections:
- removed net SPI_CS: U3.20
Changed lines of the file:
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@@
 <wire x1="45.74" y1="9.8425" x2="44.47" y2="8.5725" width="0.254" layer="16"/>
-</signal>
-<signal name="SPI_CS">
-<contactref element="U3" pad="20"/>
 </signal>
 <signal name="NSEL">

Commit message: Add files via upload
Parts:
- U3: value STM32L011 -> STM32L031K6T6
Changed lines of the file:
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@@
 </element>
 <element name="U2" library="CG2179M2" package="SOT363" value="CG2179M2" x="65.715" y="3.4925" rot="R270"/>
-<element name="U3" library="STM32L011" package="LQFP32-7X7" value="STM32L011" x="38.4175" y="8.5725"/>
+<element name="U3" library="STM32L011" package="LQFP32-7X7" value="STM32L031K6T6" x="38.4175" y="8.5725"/>
 <element name="X1" library="con-coax" package="J502-ND-142-0711-821/826" value="SMA" x="77" y="9.5" rot="R180">
 <attribute name="OC_FARNELL" value="1019328" x="77" y="9.5" size="1.778" layer="27" rot="R180" display="off"/>

Commit message: Add files via upload
Parts:
- moved C0 2.00 mm to (55.8, 12.1)
- moved C1 2.00 mm to (12.3, 3.49)
- moved C2 2.00 mm to (26.3, 10.5)
- moved C3 2.00 mm to (12.9, 16.2)
- moved C4 2.00 mm to (7.21, 3.49)
- moved C5 2.00 mm to (45.0, 4.76)
- moved C6 2.00 mm to (29.4, 13.7)
- moved C7 2.00 mm to (46.3, 14.6)
- moved C8 2.00 mm to (50.1, 14.6)
- moved CC1 2.00 mm to (60.2, 5.71)
- moved CC2 2.00 mm to (67.5, 4.45)
- moved CC3 2.00 mm to (63.7, 6.03)
- moved CM 2.00 mm to (60.2, 12.1)
- moved CM2 2.00 mm to (67.5, 8.57)
- moved CM3 2.00 mm to (68.5, 11.7)
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Routing:
- net GND: vias 141 -> 129
Other:
- board size 77 x 19 mm -> 75 x 19 mm
